Commit message: Updated with correct meshes & model

File: R2/catkin_ws/bot_description/bot.urdf.xacro (robot description, xacro)
@@ -1,12 +1,12 @@
 <?xml version="1.0"?>
 <robot name="bot" xmlns:xacro="http://www.ros.org/wiki/xacro">
-<xacro:property name="wheelRadius" value="0.0532"/>
+<xacro:property name="wheelRadius" value="0.0732"/>
 <xacro:property name="wheelLength" value="0.05575"/>
 <xacro:property name="leftWheel" value="left_wheel"/>
 <xacro:property name="rightWheel" value="right_wheel"/>
-<xacro:macro name="wheel" params="side num reflect">
+<xacro:macro name="wheel" params="side num reflect xv yv zv">
   <link name="${side}_${num}">
     <visual>
-      <origin rpy="0 3.14592 0" xyz="0 0 0"/>
+      <origin rpy="0 ${3.14592/2} 0" xyz="${xv} ${yv} ${zv}"/>
       <geometry>
 	<mesh filename="package://bot_description/meshes/wheel.dae" />
@@ -15,7 +15,7 @@
     </visual>
     <collision>
-      <geometry>
-         <cylinder length="${wheelLength}" radius="${wheelRadius}"/>
-         <origin rpy="0 ${3.14592/2} 0" xyz="0 0 0"/>
+	<origin rpy="0 ${3.14592/2} 0" xyz="${xv} ${yv} ${zv}"/>
+        <geometry>
+         <mesh filename="package://bot_description/meshes/wheel.dae" />
       </geometry>
     </collision>
@@ -26,9 +26,9 @@
 </link>
   <joint name="${side}_${num}_joint" type="continuous">
-    <axis xyz="0 0 1" />
+    <axis xyz="0.05 0 1" />
     <limit effort="10000.0" velocity="3"/>
     <parent link="base_link"/>
     <child link="${side}_${num}"/>
-    <origin rpy="0 ${3.14592/2} 0" xyz="${0.2 * reflect} ${0.3 - (0.2 * num)} -0.12"/>
+    <origin rpy="0 ${3.14592/2} 0" xyz="${0.2 * reflect} ${0.3 - (0.2 * num)} -0.10"/>
   </joint>
   <gazebo reference="${side}_${num}">
@@ -65,5 +65,5 @@
 		<parent link="base_link"/>
 		<child link="hokuyo_link"/>
-		<origin xyz="0.0 -0.13 0.25" rpy="0 0 -1.572" />
+		<origin xyz="0.0 -0.3 0.20" rpy="0 0 -1.572" />
 	</joint>
 	<gazebo reference="hokuyo_link">
@@ -108,5 +108,5 @@
         <mesh filename="package://bot_description/meshes/carfullblended.dae"/>
       </geometry>
-      <origin rpy="0 0 0" xyz="0.044112 -0.311197 -0.038199"/>
+      <origin rpy="0 0 0" xyz="-0.01 -0.05 -0.08"/>
       <material name="grey"/>
     </visual>
@@ -115,5 +115,5 @@
         <mesh filename="package://bot_description/meshes/carfullblended.dae"/>
       </geometry>
-      <origin rpy="0 0 0" xyz="0 0 0"/>
+      <origin rpy="0 0 0" xyz="-0.01 -0.05 -0.08"/>
     </collision>
   </link>
@@ -129,12 +129,12 @@
     <origin rpy="0 0 0" xyz="0 0 0"/>
   </joint>
-<xacro:wheel side="left_wheel" num="0" reflect="-1"/>
-<xacro:wheel side="left_wheel" num="1" reflect="-1"/>
-<xacro:wheel side="left_wheel" num="2" reflect="-1"/>
-<xacro:wheel side="left_wheel" num="3" reflect="-1"/>
-<xacro:wheel side="right_wheel" num="0" reflect="1"/>
-<xacro:wheel side="right_wheel" num="1" reflect="1"/>
-<xacro:wheel side="right_wheel" num="2" reflect="1"/>
-<xacro:wheel side="right_wheel" num="3" reflect="1"/>
+<xacro:wheel side="left_wheel" num="0" reflect="-1" xv="0" yv="0" zv="0.02"/>
+<xacro:wheel side="left_wheel" num="1" reflect="-1" xv="0" yv="0" zv="0.02"/>
+<xacro:wheel side="left_wheel" num="2" reflect="-1" xv="0" yv="0" zv="0.02"/>
+<xacro:wheel side="left_wheel" num="3" reflect="-1" xv="0" yv="0" zv="0.02"/>
+<xacro:wheel side="right_wheel" num="0" reflect="1" xv="0" yv="0" zv="-0.02"/>
+<xacro:wheel side="right_wheel" num="1" reflect="1" xv="0" yv="0" zv="-0.02"/>
+<xacro:wheel side="right_wheel" num="2" reflect="1" xv="0" yv="0" zv="-0.02"/>
+<xacro:wheel side="right_wheel" num="3" reflect="1" xv="0" yv="0" zv="-0.02"/>
   <gazebo>
   <plugin name="gazebo_ros_control" filename="libgazebo_ros_control.so">

File: R2/catkin_ws/bot_description/world/bot.urdf.xacro (robot description, xacro)
@@ -10,5 +10,5 @@
       <geometry>
         <cylinder length="${wheelLength}" radius="${wheelRadius}"/>
-        <origin rpy="0 3.14592/2 0" xyz="${0.2 * reflect} ${0.3 - (0.2 * num)} -0.12"/>
+        <origin rpy="0 ${3.14592/2} 0" xyz="${0.2 * reflect} ${0.3 - (0.2 * num)} -0.12"/>
       </geometry>
       <material name="Black"/>
@@ -17,5 +17,5 @@
       <geometry>
          <cylinder length="${wheelLength}" radius="${wheelRadius}"/>
-         <origin rpy="0 3.14592/2 0" xyz="${0.2 * reflect} ${0.3 - (0.2 * num)} -0.12"/>
+         <origin rpy="0 ${3.14592/2} 0" xyz="${0.2 * reflect} ${0.3 - (0.2 * num)} -0.12"/>
       </geometry>
     </collision>

Commit message: Now turning in rviz

File: R2/catkin_ws/bot_description/bot.urdf.xacro (robot description, xacro)
@@ -21,5 +21,5 @@
     </collision>
     <inertial>
-      <mass value = "1" />
+      <mass value = "0.1" />
       <inertia ixx="0.00143" ixy="0.0" ixz="0.0" iyy="0.00143" iyz="0.0" izz="0.00125"/>
     </inertial>
@@ -27,5 +27,5 @@
   <joint name="${side}_${num}_joint" type="continuous">
     <axis xyz="0.05 0 1" />
-    <limit effort="10000.0" velocity="3"/>
+    <limit effort="10000.0" velocity="100"/>
     <parent link="base_link"/>
     <child link="${side}_${num}"/>
@@ -120,5 +120,5 @@
   <link name="dummy_link">
     <inertial>
-      <mass value = "10" />
+      <mass value = "1" />
       <inertia ixx="0.05666" ixy="0.0" ixz="0.0" iyy="0.00666" iyz="0.0" izz="0.05666"/>
     </inertial>

Commit message: Using different move_base files
doesn't use amcl

File: R2/catkin_ws/bot_description/bot.urdf.xacro (robot description, xacro)
@@ -8,5 +8,5 @@
   <link name="${side}_${num}">
     <visual>
-      <origin rpy="0 ${3.14592/2} 0" xyz="${xv} ${yv} ${zv}"/>
+      <origin rpy="0 1.57079632679 0" xyz="${xv} ${yv} ${zv}"/>
       <geometry>
 	<mesh filename="package://bot_description/meshes/wheel.dae" />
@@ -15,5 +15,5 @@
     </visual>
     <collision>
-	<origin rpy="0 ${3.14592/2} 0" xyz="${xv} ${yv} ${zv}"/>
+	<origin rpy="0 1.57079632679 0" xyz="${xv} ${yv} ${zv}"/>
         <geometry>
          <mesh filename="package://bot_description/meshes/wheel.dae" />
@@ -30,5 +30,5 @@
     <parent link="base_link"/>
     <child link="${side}_${num}"/>
-    <origin rpy="0 ${3.14592/2} 0" xyz="${0.2 * reflect} ${0.3 - (0.2 * num)} -0.10"/>
+    <origin rpy="0 ${3.14592/2} 3.14159265359" xyz="${0.2 * reflect} ${0.3 - (0.2 * num)} -0.10"/>
   </joint>
   <gazebo reference="${side}_${num}">
@@ -65,5 +65,5 @@
 		<parent link="base_link"/>
 		<child link="hokuyo_link"/>
-		<origin xyz="0.0 -0.3 0.20" rpy="0 0 -1.572" />
+		<origin xyz="0.0 0.3 0.20" rpy="0 0 1.572" />
 	</joint>
 	<gazebo reference="hokuyo_link">
@@ -108,5 +108,5 @@
         <mesh filename="package://bot_description/meshes/carfullblended.dae"/>
       </geometry>
-      <origin rpy="0 0 0" xyz="-0.01 -0.05 -0.08"/>
+      <origin rpy="0 0 3.14159265359" xyz="-0.01 -0.05 -0.08"/>
       <material name="grey"/>
     </visual>
@@ -115,5 +115,5 @@
         <mesh filename="package://bot_description/meshes/carfullblended.dae"/>
       </geometry>
-      <origin rpy="0 0 0" xyz="-0.01 -0.05 -0.08"/>
+      <origin rpy="0 0 3.14159265359" xyz="-0.01 -0.05 -0.08"/>
     </collision>
   </link>
