Commit message: Perfect Trojan Horse

File: jackal.urdf.xacro (robot description, xacro)
@@ -17,9 +17,6 @@
   <material name="yellow"><color rgba="0.8 0.8 0.0 1.0" /></material>
   <material name="black"><color rgba="0.15 0.15 0.15 1.0" /></material>
-  <xacro:macro name="wheel" params="prefix *joint_pose">
+   <xacro:macro name="wheel" params="prefix *joint_pose">
     <link name="${prefix}_wheel_link">
-      <visual>
-        <origin xyz="0 0 0" rpy="${PI/2} 0 0"/>
-      </visual>
       <collision>
         <origin xyz="0 0 0" rpy="${PI/2} 0 0"/>
@@ -58,5 +55,5 @@
     </transmission>
   </xacro:macro>
-<xacro:macro name="wheel" params="side num reflect xv yv zv">
+<xacro:macro name="wheel2" params="side num reflect xv yv zv">
   <link name="${side}_${num}">
     <visual>
@@ -67,13 +64,7 @@
       <material name="Grey"/>
     </visual>
-    <collision>
-	<origin rpy="0 1.57079632679 0" xyz="${xv} ${yv} ${zv}"/>
-        <geometry>
-         <mesh filename="package://bot_description/meshes/wheel.dae" />
-      </geometry>
-    </collision>
     <inertial>
       <mass value = "0.1" />
-      <inertia ixx="0.00143" ixy="0.0" ixz="0.0" iyy="0.00143" iyz="0.0" izz="0.00125"/>
+      <inertia ixx="0.0" ixy="0.0" ixz="0.0" iyy="0.0" iyz="0.0" izz="0.0"/>
     </inertial>
 </link>
@@ -83,5 +74,5 @@
     <parent link="base_link"/>
     <child link="${side}_${num}"/>
-    <origin rpy="0 ${3.14592/2} 3.14159265359" xyz="${0.2 * reflect} ${0.3 - (0.2 * num)} -0.10"/>
+    <origin rpy="0 ${3.14592/2} 1.57079632679" xyz="${0.3 - (0.2 * num)} ${0.2 * reflect} 0.01"/>
   </joint>
   <gazebo reference="${side}_${num}">
@@ -105,12 +96,12 @@
     <origin xyz="${-wheelbase/2} ${-track/2} ${wheel_vertical_offset}" rpy="0 0 0" />
   </xacro:wheel>
-<xacro:wheel side="left_wheel" num="0" reflect="-1" xv="0" yv="0" zv="0.02"/>
-<xacro:wheel side="left_wheel" num="1" reflect="-1" xv="0" yv="0" zv="0.02"/>
-<xacro:wheel side="left_wheel" num="2" reflect="-1" xv="0" yv="0" zv="0.02"/>
-<xacro:wheel side="left_wheel" num="3" reflect="-1" xv="0" yv="0" zv="0.02"/>
-<xacro:wheel side="right_wheel" num="0" reflect="1" xv="0" yv="0" zv="-0.02"/>
-<xacro:wheel side="right_wheel" num="1" reflect="1" xv="0" yv="0" zv="-0.02"/>
-<xacro:wheel side="right_wheel" num="2" reflect="1" xv="0" yv="0" zv="-0.02"/>
-<xacro:wheel side="right_wheel" num="3" reflect="1" xv="0" yv="0" zv="-0.02"/>
+<xacro:wheel2 side="left_wheel" num="0" reflect="-1" xv="0" yv="0" zv="0.02"/>
+<xacro:wheel2 side="left_wheel" num="1" reflect="-1" xv="0" yv="0" zv="0.02"/>
+<xacro:wheel2 side="left_wheel" num="2" reflect="-1" xv="0" yv="0" zv="0.02"/>
+<xacro:wheel2 side="left_wheel" num="3" reflect="-1" xv="0" yv="0" zv="0.02"/>
+<xacro:wheel2 side="right_wheel" num="0" reflect="1" xv="0" yv="0" zv="-0.02"/>
+<xacro:wheel2 side="right_wheel" num="1" reflect="1" xv="0" yv="0" zv="-0.02"/>
+<xacro:wheel2 side="right_wheel" num="2" reflect="1" xv="0" yv="0" zv="-0.02"/>
+<xacro:wheel2 side="right_wheel" num="3" reflect="1" xv="0" yv="0" zv="-0.02"/>
   <link name="base_link"></link>
   <joint name="base_link_joint" type="fixed">
@@ -121,5 +112,5 @@
   <link name="chassis_link">
     <visual>
-      <origin xyz="0 0 ${footprint_vertical_offset}" rpy="${PI/2} 0 ${PI/2}"/>
+      <origin rpy="0 0 4.71238898039" xyz="-0.01 0 0.01"/>
       <geometry>
         <mesh filename="package://jackal_description/meshes/carfullblended.dae"/>
@@ -128,5 +119,5 @@
     </visual>
     <collision>
-      <origin xyz="0 0 ${chassis_height/2}"/>
+      <origin rpy="0 0 4.71238898039" xyz="-0.01 0 0"/>
       <geometry>
          <mesh filename="package://jackal_description/meshes/carfullblended.dae"/>
@@ -146,17 +137,8 @@
   <xacro:unless value="$(optenv JACKAL_FRONT_ACCESSORY_FENDER 0)">
     <link name="front_fender_link">
-      <visual>
-        <material name="yellow" />
-      </visual>
     </link>
   </xacro:unless>
   <xacro:if value="$(optenv JACKAL_FRONT_ACCESSORY_FENDER 0)">
     <link name="front_fender_link">
-      <visual>
-        <geometry>
-          <mesh filename="package://jackal_description/meshes/accessory_fender.stl"/>
-        </geometry>
-        <material name="yellow" />
-      </visual>
     </link>
     <link name="front_fender_accessory_link"/>
@@ -174,20 +156,8 @@
   <xacro:unless value="$(optenv JACKAL_REAR_ACCESSORY_FENDER 0)">
     <link name="rear_fender_link">
-      <visual>
-        <geometry>
-          <mesh filename="package://jackal_description/meshes/jackal-fender.stl"/>
-        </geometry>
-        <material name="yellow" />
-      </visual>
     </link>
   </xacro:unless>
   <xacro:if value="$(optenv JACKAL_REAR_ACCESSORY_FENDER 0)">
     <link name="rear_fender_link">
-      <visual>
-        <geometry>
-          <mesh filename="package://jackal_description/meshes/accessory_fender.stl"/>
-        </geometry>
-        <material name="yellow" />
-      </visual>
     </link>
     <link name="rear_fender_accessory_link"/>

Commit message: thig

File: jackal.urdf.xacro (robot description, xacro)
@@ -60,5 +60,5 @@
       <origin rpy="0 1.57079632679 0" xyz="${xv} ${yv} ${zv}"/>
       <geometry>
-	<mesh filename="package://bot_description/meshes/wheel.dae" />
+	<mesh filename="package://jackal_description/meshes/wheel.dae" />
       </geometry>
       <material name="Grey"/>

Commit message: jackal 2

File: jackal.urdf.xacro (robot description, xacro)
@@ -74,5 +74,5 @@
     <parent link="base_link"/>
     <child link="${side}_${num}"/>
-    <origin rpy="0 ${3.14592/2} 1.57079632679" xyz="${0.3 - (0.2 * num)} ${0.2 * reflect} 0.01"/>
+    <origin rpy="0 ${3.14592/2} 1.57079632679" xyz="${0.3 - (0.2 * num)} ${(0.2 * reflect) + 0.1} 0.01"/>
   </joint>
   <gazebo reference="${side}_${num}">
@@ -104,7 +104,45 @@
 <xacro:wheel2 side="right_wheel" num="2" reflect="1" xv="0" yv="0" zv="-0.02"/>
 <xacro:wheel2 side="right_wheel" num="3" reflect="1" xv="0" yv="0" zv="-0.02"/>
+<link name="hokuyo_link">
+        <visual>
+			    <origin rpy="0 0 0" xyz="0 0 0"/>
+			    <material name="blue"/>
+        </visual>
+    </link>
+	<joint name="hokuyo_joint" type="fixed">
+		<parent link="base_link"/>
+		<child link="hokuyo_link"/>
+		<origin xyz="0.22 0.1 0.31" rpy="0 0 0" />
+	</joint>
+	<gazebo reference="hokuyo_link">
+    <material>Gazebo/White</material>
+	    <sensor name="head_hokuyo_sensor" type="ray">
+	      <pose>0.05 0 0 0 0 0</pose>
+	      <visualize>true</visualize>
+	      <update_rate>40</update_rate>
+	      <ray>
+	        <scan>
+	          <horizontal>
+	            <samples>720</samples>
+	            <resolution>1</resolution>
+	            <min_angle>-1.570796</min_angle>
+	            <max_angle>1.570796</max_angle>
+	          </horizontal>
+	        </scan>
+	        <range>
+	          <min>0.10</min>
+	          <max>10.0</max>
+	          <resolution>0.001</resolution>
+	        </range>
+	      </ray>
+	      <plugin filename="libgazebo_ros_laser.so" name="gazebo_ros_head_hokuyo_controller">
+	        <topicName>/scan</topicName>
+	        <frameName>hokuyo_link</frameName>
+	      </plugin>
+	    </sensor>
+  	</gazebo>
   <link name="base_link"></link>
   <joint name="base_link_joint" type="fixed">
-    <origin xyz="0 0 0" rpy="0 0 0" />
+    <origin xyz="0.1 0.1 0" rpy="0 0 0" />
     <parent link="base_link"/>
     <child link="chassis_link" />
@@ -112,5 +150,5 @@
   <link name="chassis_link">
     <visual>
-      <origin rpy="0 0 4.71238898039" xyz="-0.01 0 0.01"/>
+      <origin rpy="0 0 1.57079632679" xyz="-0.01 0 0.01"/>
       <geometry>
         <mesh filename="package://jackal_description/meshes/carfullblended.dae"/>
@@ -119,5 +157,5 @@
     </visual>
     <collision>
-      <origin rpy="0 0 4.71238898039" xyz="-0.01 0 0"/>
+       <origin rpy="0 0 1.57079632679" xyz="-0.01 0 0.01"/>
       <geometry>
          <mesh filename="package://jackal_description/meshes/carfullblended.dae"/>
@@ -191,7 +229,4 @@
   <link name="navsat_link">
     <visual>
-      <geometry>
-        <cylinder radius="0.026" length="0.016" />
-      </geometry>
       <origin xyz="0 0 0.008" />
       <material name="black" />
