Commit message: Final 16.04 Update

File: bot_description/bot.urdf.xacro (robot description, xacro)
@@ -21,12 +21,12 @@
     </collision>
     <inertial>
-      <mass value = "0.1" />
-      <inertia ixx="0.00143" ixy="0.0" ixz="0.0" iyy="0.00143" iyz="0.0" izz="0.00125"/>
+      <mass value = "1" />
+      <inertia ixx="0.0017583" ixy="0.0" ixz="0.0" iyy="0.0017583" iyz="0.0" izz="0.00245"/>
     </inertial>
 </link>
   <link name="${side}_${num}_dummy">
     <inertial>
-      <mass value = "0.1" />
-      <inertia ixx="0.00143" ixy="0.0" ixz="0.0" iyy="0.00143" iyz="0.0" izz="0.00125"/>
+      <mass value = "0.6" />
+      <inertia ixx="0.001" ixy="0.0" ixz="0.0" iyy="0.001" iyz="0.0" izz="0.001"/>
     </inertial>
   </link>
@@ -36,5 +36,5 @@
     <parent link="base_link"/>
     <child link="${side}_${num}_dummy"/>
-    <origin rpy="0 0 0" xyz="${0.3 - (0.2 * num)} ${0.2 * reflect}  -0.10"/>
+    <origin rpy="0 0 0" xyz="${0.3 - (0.2 * num)} ${0.2 * reflect}  0.1"/>
   </joint>
   <transmission name="${side}_${num}_trans2">
@@ -73,8 +73,8 @@
         <visual>
 			<origin rpy="0 0 0" xyz="0 0 0"/>
-            <geometry>
-                <box size="0.1 0.1 0.1"/>
-            </geometry>
 			<material name="blue"/>
+        <geometry>
+          		<cylinder length="0.001" radius="0.001"/>
+        </geometry>
         </visual>
     </link>
@@ -82,29 +82,29 @@
 		<parent link="base_link"/>
 		<child link="hokuyo_link"/>
-		<origin xyz="0.0 0.0 0.30" rpy="0 0 0" />
+		<origin xyz="0.0 0.0 0.48" rpy="0 0 0" />
 	</joint>
 	<gazebo reference="hokuyo_link">
-    <material>Gazebo/White</material>
+          <material>Gazebo/White</material>
 	    <sensor name="head_hokuyo_sensor" type="ray">
 	      <pose>0.05 0 0 0 0 0</pose>
-	      <visualize>true</visualize>
+	      <visualize>false</visualize>
 	      <update_rate>40</update_rate>
 	      <ray>
 	        <scan>
 	          <horizontal>
-	            <samples>720</samples>
+	            <samples>1440</samples>
 	            <resolution>1</resolution>
-	            <min_angle>-1.570796</min_angle>
-	            <max_angle>1.570796</max_angle>
+	            <min_angle>-3.141592</min_angle>
+	            <max_angle>3.141592</max_angle>
 	          </horizontal>
 	        </scan>
 	        <range>
 	          <min>0.10</min>
-	          <max>10.0</max>
+	          <max>25.0</max>
 	          <resolution>0.001</resolution>
 	        </range>
 	      </ray>
 	      <plugin filename="libgazebo_ros_laser.so" name="gazebo_ros_head_hokuyo_controller">
-	        <topicName>/scan</topicName>
+	        <topicName>/bot/scan</topicName>
 	        <frameName>hokuyo_link</frameName>
 	      </plugin>
@@ -120,30 +120,25 @@
     <color rgba="0 0 0 1"/>
   </material>
+<!-- ======================= ECV Model & Meshes =============================== -->
   <link name="base_link">
     <visual>
       <geometry>
-        <mesh filename="package://bot_description/meshes/carfullblended.dae"/>
+        <mesh filename="package://bot_description/meshes/TrueECV.dae"/>
       </geometry>
-      <origin rpy="0 0 1.5712645" xyz="-0.01 -0.007 -0.08"/>
+      <origin rpy="0 0 1.5712645" xyz="0.02 -0.007 0.31"/>
       <material name="white"/>
     </visual>
     <collision>
       <geometry>
-        <mesh filename="package://bot_description/meshes/carfullblended.dae"/>
+          <box size="0.4 1.0 0.3"/>
       </geometry>
-      <origin rpy="0 0 1.5712645" xyz="-0.01 -0.007 -0.08"/>
+      <origin rpy="0 0 1.5712645" xyz="0.02 -0.007 0.31"/>
     </collision>
-  </link>
-  <link name="dummy_link">
     <inertial>
+      <origin rpy="0 0 0" xyz="0.02 -0.007 0.31"/>
       <mass value = "1" />
-      <inertia ixx="0.05666" ixy="0.0" ixz="0.0" iyy="0.00666" iyz="0.0" izz="0.05666"/>
+      <inertia ixx="0.0208" ixy="0.0" ixz="0.0" iyy="0.097" iyz="0.0" izz="0.097"/>
     </inertial>
   </link>
-  <joint name="dummy_joint" type="fixed">
-    <parent link="base_link"/>
-    <child link="dummy_link"/>
-    <origin rpy="0 0 0" xyz="0 0 0"/>
-  </joint>
 <xacro:wheel side="left_wheel" num="0" reflect="1" xv="0" yv="0" zv="0.02"/>
 <xacro:wheel side="left_wheel" num="1" reflect="1" xv="0" yv="0" zv="0.02"/>
